Commit message: Update ARM URDF

File: urdf/arm.urdf (robot description, URDF)
Before this commit: robot zebra_zero, 8 links, 7 joints
Links:
- link base_link: geometry collision cylinder length=0.5 radius=0.05; visual box size=0.3 0.1 0.6
- link fifth_link: geometry collision cylinder length=0.5 radius=0.05; visual mesh filename=ZebraLinkThree.stl scale=0.01 0.01 0.01
- link first_link: geometry collision box size=0.35 0.7 0.7; visual mesh filename=ZebraBase.stl scale=0.01 0.01 0.01
- link fourth_link: geometry collision cylinder length=0.5 radius=0.05; visual cylinder length=0.05 radius=0.075
- link second_link: geometry collision cylinder length=0.35 radius=0.05; visual mesh filename=ZebraLinkOne.stl scale=0.01 0.01 0.01
- link sixth_link: geometry collision cylinder length=0.1 radius=0.05; visual cylinder length=0.05 radius=0.075
- link third_link: geometry collision mesh filename=ZebraLinkTwo.stl scale=0.01 0.01 0.01; visual mesh filename=ZebraLinkTwo.stl scale=0.01 0.01 0.01
Joints:
- joint fifth_joint: limit lower=-2.2 upper=0.7 effort=30 velocity=1.0 -> lower=-2.2 upper=2.2 effort=30 velocity=1.0; origin xyz=0 0 0.1 rpy=0 0 0 -> xyz=0 0 0.05 rpy=0 0 0
- joint fourth_joint: origin xyz=0 0 0.35 rpy=0 0 0 -> xyz=0 0 0.45 rpy=0 0 0
- joint second_joint: origin xyz=0 0 0.25 rpy=0 0 0 -> xyz=0 0 0.45 rpy=0 0 0
- joint third_joint: origin xyz=0 0 0.35 rpy=0 0 0 -> xyz=0 0 0.60 rpy=0 0 0

Commit message: Cleanups

File: urdf/arm.urdf (robot description, URDF)
Before this commit: robot zebra_zero, 8 links, 7 joints
Links:
- link fifth_link: geometry collision cylinder length=0.5 radius=0.05; visual mesh filename=package://zebra_zero/urdf/ZebraLinkThree.stl scale=0.01 0.01 0.01
- link first_link: geometry collision box size=0.35 0.7 0.7; visual mesh filename=package://zebra_zero/urdf/ZebraBase.stl scale=0.01 0.01 0.01
- link second_link: geometry collision cylinder length=0.35 radius=0.05; visual mesh filename=package://zebra_zero/urdf/ZebraLinkOne.stl scale=0.01 0.01 0.01
- link third_link: geometry collision mesh filename=ZebraLinkTwo.stl scale=0.01 0.01 0.01; visual mesh filename=package://zebra_zero/urdf/ZebraLinkTwo.stl scale=0.01 0.01 0.01

Commit message: Updates to URDF

File: urdf/arm.urdf (robot description, URDF)
Before this commit: robot zebra_zero, 8 links, 7 joints
Links:
- link third_link: geometry collision mesh filename=package://zebra_zero/urdf/ZebraLinkTwo.stl scale=0.01 0.01 0.01; visual mesh filename=package://zebra_zero/urdf/ZebraLinkTwo.stl scale=0.01 0.01 0.01
Joints:
- joint second_joint: limit lower=-2.2 upper=0.7 effort=30 velocity=1.0 -> lower=-0.7 upper=2.2 effort=30 velocity=1.0
- joint third_joint: axis 0 1 0 -> 0 -1 0

Commit message: Improve URDF

File: urdf/arm.urdf (robot description, URDF)
Before this commit: robot zebra_zero, 8 links, 7 joints
Links:
- link base_link: geometry collision cylinder length=0.5 radius=0.05; visual box size=0.15 0.04 0.3
- link fifth_link: geometry collision cylinder length=0.25 radius=0.025; visual mesh filename=package://zebra_zero/urdf/ZebraLinkThree.stl scale=0.005 0.005 0.005
- link first_link: geometry collision box size=0.35 0.7 0.7; visual mesh filename=package://zebra_zero/urdf/ZebraBase.stl scale=0.005 0.005 0.005
- link fourth_link: geometry collision cylinder length=0.25 radius=0.025; visual cylinder length=0.025 radius=0.0375
- link second_link: geometry collision cylinder length=0.35 radius=0.05; visual mesh filename=package://zebra_zero/urdf/ZebraLinkOne.stl scale=0.005 0.005 0.005
- link sixth_link: geometry collision cylinder length=0.05 radius=0.025; visual cylinder length=0.025 radius=0.0375
- link third_link: geometry collision mesh filename=package://zebra_zero/urdf/ZebraLinkTwo.stl scale=0.005 0.005 0.005; visual mesh filename=package://zebra_zero/urdf/ZebraLinkTwo.stl scale=0.005 0.005 0.005
Joints:
- joint fifth_joint: origin xyz=0 0 0.05 rpy=0 0 0 -> xyz=0 0 0.045 rpy=0 0 0
- joint first_joint: origin xyz=0 0 0 rpy=1.57 0 0 -> xyz=0 -0.045 0 rpy=1.57 0 0
- joint fourth_joint: origin xyz=0 0 0.45 rpy=0 0 0 -> xyz=0 0 0.1925 rpy=0 0 0
- joint second_joint: origin xyz=0 0 0.45 rpy=0 0 0 -> xyz=0 0 0.24 rpy=0 0 0
- joint sixth_joint: origin xyz=0 0 0.1 rpy=0 0 0 -> xyz=0 0 0.04 rpy=0 0 0
- joint third_joint: origin xyz=0 0 0.60 rpy=0 0 0 -> xyz=0 0 0.30 rpy=0 0 0

Commit message: Add a couple scripts, fix joint limits

File: urdf/arm.urdf (robot description, URDF)
Before this commit: robot zebra_zero, 8 links, 7 joints
Joints:
- joint fifth_joint: limit lower=-2.2 upper=2.2 effort=30 velocity=1.0 -> lower=-1.6 upper=1.6 effort=30 velocity=1.0
- joint first_joint: limit lower=-2.2 upper=0.7 effort=30 velocity=1.0 -> lower=-3.14 upper=3.14 effort=30 velocity=1.0
- joint fourth_joint: limit lower=-2.2 upper=0.7 effort=30 velocity=1.0 -> lower=-3.14 upper=3.14 effort=30 velocity=1.0
- joint second_joint: limit lower=-0.7 upper=2.2 effort=30 velocity=1.0 -> lower=-0.2 upper=2.2 effort=30 velocity=1.0
- joint sixth_joint: limit lower=-2.2 upper=0.7 effort=30 velocity=1.0 -> lower=-3.14 upper=3.14 effort=30 velocity=1.0
- joint third_joint: limit lower=-2.2 upper=0.7 effort=30 velocity=1.0 -> lower=-1.6 upper=0.4 effort=30 velocity=1.0

Commit message: Fix up collision geometry

File: urdf/arm.urdf (robot description, URDF)
Before this commit: robot zebra_zero, 8 links, 7 joints
Links:
- link base_link: geometry collision box size=0.15 0.04 0.3; visual box size=0.15 0.04 0.3
- link fifth_link: geometry collision mesh filename=package://zebra_zero/urdf/ZebraLinkThree.stl scale=0.005 0.005 0.005; visual mesh filename=package://zebra_zero/urdf/ZebraLinkThree.stl scale=0.005 0.005 0.005
- link first_link: geometry collision mesh filename=package://zebra_zero/urdf/ZebraBase.stl scale=0.005 0.005 0.005; visual mesh filename=package://zebra_zero/urdf/ZebraBase.stl scale=0.005 0.005 0.005
- link fourth_link: geometry collision cylinder length=0.025 radius=0.0375; visual cylinder length=0.025 radius=0.0375
- link second_link: geometry collision mesh filename=package://zebra_zero/urdf/ZebraLinkOne.stl scale=0.005 0.005 0.005; visual mesh filename=package://zebra_zero/urdf/ZebraLinkOne.stl scale=0.005 0.005 0.005
- link sixth_link: geometry collision cylinder length=0.025 radius=0.0375; visual cylinder length=0.025 radius=0.0375
