Commit message: Start moving to xacro, add support for mock components

File: urdf/arm.urdf.xacro (robot description, xacro)
@@ -1,3 +1,14 @@
-<robot name="zebra_zero">
+<?xml version="1.0"?>
+<robot xmlns:xacro="http://www.ros.org/wiki/xacro" name="zebra_zero">
+  <xacro:arg name="ros2_control_hardware_type" default="zebra" />
+  <xacro:macro name="ros2_control" params="ros2_control_hardware_type">
+    <xacro:if value="${ros2_control_hardware_type == 'mock_components'}">
+      <plugin>mock_components/GenericSystem</plugin>
+      <param name="calculate_dynamics">true</param>
+    </xacro:if>
+    <xacro:if value="${ros2_control_hardware_type == 'zebra'}">
+      <plugin>zebra_zero/RobotSystem</plugin>
+    </xacro:if>
+  </xacro:macro>
   <link name="base_link">
     <visual>
@@ -180,5 +191,5 @@
   <ros2_control name="zebra_zero" type="system">
     <hardware>
-      <plugin>zebra_zero/RobotSystem</plugin>
+      <xacro:ros2_control ros2_control_hardware_type="$(arg ros2_control_hardware_type)" />
     </hardware>
     <joint name="first_joint">

Commit message: Update joint limits to match ros2 control

File: urdf/arm.urdf.xacro (robot description, xacro)
@@ -87,5 +87,5 @@
     <origin rpy="0 0 0" xyz="0 0 0.24"/>
     <axis xyz="0 1 0"/>
-    <limit effort="30" velocity="1.0" lower="-0.2" upper="2.2" />
+    <limit effort="30" velocity="1.0" lower="-1.07" upper="0.5" />
   </joint>
   <link name="third_link">
@@ -112,5 +112,5 @@
     <origin rpy="0 0 0" xyz="0 0 0.30"/>
     <axis xyz="0 -1 0"/>
-    <limit effort="30" velocity="1.0" lower="-1.6" upper="0.4" />
+    <limit effort="30" velocity="1.0" lower="-1.07" upper="1.57" />
   </joint>
   <link name="fourth_link">
@@ -162,5 +162,5 @@
     <origin rpy="0 0 0" xyz="0 0 0.045"/>
     <axis xyz="0 1 0"/>
-    <limit effort="30" velocity="1.0" lower="-1.6" upper="1.6" />
+    <limit effort="30" velocity="1.0" lower="-3.14" upper="3.14" />
   </joint>
   <link name="sixth_link">

Commit message: Updates for joint limits

File: urdf/arm.urdf.xacro (robot description, xacro)
@@ -87,5 +87,5 @@
     <origin rpy="0 0 0" xyz="0 0 0.24"/>
     <axis xyz="0 1 0"/>
-    <limit effort="30" velocity="1.0" lower="-1.07" upper="0.5" />
+    <limit effort="30" velocity="1.0" lower="-1.07" upper="1.6" />
   </joint>
   <link name="third_link">
@@ -112,5 +112,5 @@
     <origin rpy="0 0 0" xyz="0 0 0.30"/>
     <axis xyz="0 -1 0"/>
-    <limit effort="30" velocity="1.0" lower="-1.07" upper="1.57" />
+    <limit effort="30" velocity="1.0" lower="-1.6" upper="1.07" />
   </joint>
   <link name="fourth_link">
@@ -233,8 +233,8 @@
       </state_interface>
     </joint>
-      <joint name="third_joint">
-      <command_interface name="position">
-        <param name="min">-1.07</param>
-        <param name="max">1.57</param>
+    <joint name="third_joint">
+      <command_interface name="position">
+        <param name="min">-1.6</param>
+        <param name="max">1.07</param>
       </command_interface>
       <command_interface name="velocity">

Commit message: Updates for joint limits

File: urdf/arm.urdf.xacro (robot description, xacro)
@@ -87,5 +87,5 @@
     <origin rpy="0 0 0" xyz="0 0 0.24"/>
     <axis xyz="0 1 0"/>
-    <limit effort="30" velocity="1.0" lower="-1.07" upper="1.6" />
+    <limit effort="30" velocity="1.0" lower="-1.07" upper="1.7" />
   </joint>
   <link name="third_link">
@@ -112,5 +112,5 @@
     <origin rpy="0 0 0" xyz="0 0 0.30"/>
     <axis xyz="0 -1 0"/>
-    <limit effort="30" velocity="1.0" lower="-1.6" upper="1.07" />
+    <limit effort="30" velocity="1.0" lower="-1.7" upper="1.07" />
   </joint>
   <link name="fourth_link">
@@ -216,5 +216,5 @@
       <command_interface name="position">
         <param name="min">-1.07</param>
-        <param name="max">1.6</param>
+        <param name="max">1.7</param>
       </command_interface>
       <command_interface name="velocity">
@@ -235,5 +235,5 @@
     <joint name="third_joint">
       <command_interface name="position">
-        <param name="min">-1.6</param>
+        <param name="min">-1.7</param>
         <param name="max">1.07</param>
       </command_interface>
